File: schematics/magic-curtains/magic-curtains.sch (KiCad schematic (older format))
At the start: 6 parts

Commit message: Undo commit and replace old files with the most recent changes.
Parts:
- added R2, R3: 10k, symbol Device:R
- renumbered Control to Control1, Crystal to Crystal1
Connections:
- net labels added: D10, D11, D12, D13, D2, D3, D4, D5, D6, D7, D8, D9, RX, TX
- wire segments 41 -> 51
Other:
- note added: "Curtain 1 Down (OPEN)"
- note added: "Curtain 1 Up (CLOSE)"
- note added: "Curtain 2 Down (OPEN)"
- note added: "Curtain 2 Up (CLOSE)"
Changed lines of the file:
@@
 $EndDescr
 $Comp
-L Device:Crystal Crystal
+L Device:Crystal Crystal1
 U 1 1 5F5A2950
 P 4100 3550
-F 0 "Crystal" V 4054 3681 50  0000 L CNN
+F 0 "Crystal1" V 4054 3681 50  0000 L CNN
 F 1 "16Mhz" V 4145 3681 50  0000 L CNN
 F 2 "" H 4100 3550 50  0001 C CNN
@@
 $EndComp
 $Comp
-L power:+5V #PWR?
+L power:+5V #PWR0101
 U 1 1 5F5A820A
 P 950 1750
-F 0 "#PWR?" H 950 1600 50  0001 C CNN
+F 0 "#PWR0101" H 950 1600 50  0001 C CNN
 F 1 "+5V" H 965 1923 50  0000 C CNN
 F 2 "" H 950 1750 50  0001 C CNN
@@
 $EndComp
 $Comp
-L power:GND #PWR?
+L power:GND #PWR0102
 U 1 1 5F5CF4DB
 P 1350 1750
-F 0 "#PWR?" H 1350 1500 50  0001 C CNN
+F 0 "#PWR0102" H 1350 1500 50  0001 C CNN
 F 1 "GND" H 1355 1577 50  0000 C CNN
 F 2 "" H 1350 1750 50  0001 C CNN
@@
 Connection ~ 3200 6200
 Wire Wire Line
-	3200 6200 5550 6200
+	3200 6200 4150 6200
 Wire Wire Line
 	3200 5750 3200 2550
@@
 	2500 2550 2500 2600
 $Comp
-L MCU_Microchip_ATmega:ATmega328P-PU Control
+L MCU_Microchip_ATmega:ATmega328P-PU Control1
 U 1 1 5F5BF002
 P 2400 4100
-F 0 "Control" H 1756 4146 50  0000 R CNN
+F 0 "Control1" H 1756 4146 50  0000 R CNN
 F 1 "ATmega328P-PU" H 1756 4055 50  0000 R CNN
 F 2 "Package_DIP:DIP-28_W7.62mm" H 2400 4100 50  0001 C CIN
@@
 	950  1750 950  2300
 Wire Wire Line
-	3150 3800 3650 3800
-Wire Wire Line
-	3650 3800 3650 2250
-Wire Wire Line
-	3150 3900 3750 3900
-Wire Wire Line
-	3750 3900 3750 2350
-Wire Wire Line
-	3750 2350 6500 2350
-Text Notes 6450 2250 2    39   Italic 0
+	3800 5850 4500 5850
+Text Notes 6500 5750 2    39   Italic 0
 Curtain Down (OPEN)
-Text Notes 6400 2350 2    39   Italic 0
+Text Notes 6450 5850 2    39   Italic 0
 Curtain Up (CLOSE)
-Wire Wire Line
-	3650 2250 6500 2250
+Wire Notes Line
+	2350 5350 2350 4550
+Wire Notes Line
+	2350 5350 2900 5350
+Text GLabel 3000 4600 2    39   Input Italic 0
+RX
+Text GLabel 3000 4700 2    39   Input Italic 0
+TX
+Text GLabel 3000 4800 2    39   Input Italic 0
+D2
+Text GLabel 3000 4900 2    39   Input Italic 0
+D3
+Text GLabel 3000 5000 2    39   Input Italic 0
+D4
+Text GLabel 3000 5100 2    39   Input Italic 0
+D5
+Text GLabel 3000 5200 2    39   Input Italic 0
+D6
+Text GLabel 3000 5300 2    39   Input Italic 0
+D7
+Text GLabel 3000 2900 2    39   Input Italic 0
+D8
+Text GLabel 3000 3000 2    39   Input Italic 0
+D9
+Text GLabel 3000 3100 2    39   Input Italic 0
+D10
+Text GLabel 3000 3200 2    39   Input Italic 0
+D11
+Text GLabel 3000 3300 2    39   Input Italic 0
+D12
+Text GLabel 3000 3400 2    39   Input Italic 0
+D13
+Wire Notes Line
+	2900 4550 2350 4550
+Wire Notes Line
+	2900 2850 2550 2850
+Wire Notes Line
+	2550 2850 2550 3450
+Wire Notes Line
+	2550 3450 2900 3450
+Wire Wire Line
+	3150 5100 6550 5100
+Wire Wire Line
+	3150 5000 6550 5000
+Wire Wire Line
+	3150 4900 6550 4900
+Wire Wire Line
+	3150 4800 6550 4800
+Text Notes 6300 4900 2    39   Italic 0
+Curtain 1 Up (CLOSE)
+Text Notes 6350 4800 2    39   Italic 0
+Curtain 1 Down (OPEN)
+Text Notes 6350 5000 2    39   Italic 0
+Curtain 2 Down (OPEN)
+Text Notes 6300 5100 2    39   Italic 0
+Curtain 2 Up (CLOSE)
+$Comp
+L Device:R R3
+U 1 1 5F63BC9B
+P 4500 6050
+F 0 "R3" H 4430 6004 50  0000 R CNN
+F 1 "10k" H 4430 6095 50  0000 R CNN
+F 2 "" V 4430 6050 50  0001 C CNN
+F 3 "~" H 4500 6050 50  0001 C CNN
+	1    4500 6050
+	-1   0    0    1
+$EndComp
+$Comp
+L Device:R R2
+U 1 1 5F63F6CA
+P 4150 6050
+F 0 "R2" H 4080 6004 50  0000 R CNN
+F 1 "10k" H 4080 6095 50  0000 R CNN
+F 2 "" V 4080 6050 50  0001 C CNN
+F 3 "~" H 4150 6050 50  0001 C CNN
+	1    4150 6050
+	-1   0    0    1
+$EndComp
+Wire Wire Line
+	3800 5850 3800 3900
+Wire Wire Line
+	3150 3900 3800 3900
+Wire Wire Line
+	6550 5750 4150 5750
+Wire Wire Line
+	3900 5750 3900 3800
+Wire Wire Line
+	3150 3800 3900 3800
+Connection ~ 4150 6200
+Wire Wire Line
+	4150 6200 4500 6200
+Connection ~ 4500 6200
+Wire Wire Line
+	4500 6200 5550 6200
+Wire Wire Line
+	4150 5900 4150 5750
+Connection ~ 4150 5750
+Wire Wire Line
+	4150 5750 3900 5750
+Wire Wire Line
+	4500 5900 4500 5850
+Connection ~ 4500 5850
+Wire Wire Line
+	4500 5850 6550 5850
 $EndSCHEMATC
