File: schematics/magic-curtains/magic-curtains.sch (KiCad schematic (older format))
At the start: 24 parts

Commit message: Doing PCB.
Parts:
- C1, C2: footprint (none) -> Capacitor_THT:CP_Radial_Tantal_D6.0mm_P5.00mm
- C3: footprint (none) -> Capacitor_THT:CP_Radial_D10.0mm_P5.00mm
- Crystal1: footprint (none) -> Crystal:Crystal_SMD_HC49-SD_HandSoldering
- GND_1, GND_2, GND_3, GND_4, INPUT_1, INPUT_2, OUTPUT_1, OUTPUT_2: footprint (none) -> Connector_Pin:Pin_D1.3mm_L11.0mm
- OUTPUT_3: renamed from OUTPUT_1; footprint (none) -> Connector_Pin:Pin_D1.3mm_L11.0mm
- OUTPUT_4: renamed from OUTPUT_2; footprint (none) -> Connector_Pin:Pin_D1.3mm_L11.0mm
- OUTPUT_5: renamed from OUTPUT_3; footprint (none) -> Connector_Pin:Pin_D1.3mm_L11.0mm
- OUTPUT_6: renamed from OUTPUT_4; footprint (none) -> Connector_Pin:Pin_D1.3mm_L11.0mm
- R1, R2, R3, R4, R5, R6, R7: footprint (none) -> Resistor_THT:R_Axial_DIN0207_L6.3mm_D2.5mm_P10.16mm_Horizontal
Changed lines of the file:
@@
 F 0 "Crystal1" V 3754 2681 50  0000 L CNN
 F 1 "16Mhz" V 3845 2681 50  0000 L CNN
-F 2 "" H 3800 2550 50  0001 C CNN
+F 2 "Crystal:Crystal_SMD_HC49-SD_HandSoldering" H 3800 2550 50  0001 C CNN
 F 3 "~" H 3800 2550 50  0001 C CNN
 	1    3800 2550
@@
 F 0 "R1" H 3120 1346 50  0000 L CNN
 F 1 "10k" H 3120 1255 50  0000 L CNN
-F 2 "" V 2980 1300 50  0001 C CNN
+F 2 "Resistor_THT:R_Axial_DIN0207_L6.3mm_D2.5mm_P10.16mm_Horizontal" V 2980 1300 50  0001 C CNN
 F 3 "~" H 3050 1300 50  0001 C CNN
 	1    3050 1300
@@
 	-1   0    0    1
 $EndComp
-Wire Wire Line
-	2100 4550 2100 4600
-Connection ~ 2100 4600
-Wire Wire Line
-	2100 4600 2100 5200
 Wire Wire Line
 	2700 2500 3500 2500
@@
 Wire Notes Line
 	2250 2450 2600 2450
-Wire Wire Line
-	2850 3800 6250 3800
 Text Notes 7100 3800 2    39   Italic 0
 Curtain 1 Up (CLOSE)
@@
 Text Notes 7100 4400 2    39   Italic 0
 Curtain 2 Up (CLOSE)
-Wire Wire Line
-	2850 2900 3500 2900
-Wire Wire Line
-	2850 2800 3600 2800
 Text GLabel 2700 2400 2    39   Input Italic 0
 D13
@@
 F 0 "R4" V 7707 3500 50  0000 C CNN
 F 1 "1k" V 7616 3500 50  0000 C CNN
-F 2 "" V 7430 3500 50  0001 C CNN
+F 2 "Resistor_THT:R_Axial_DIN0207_L6.3mm_D2.5mm_P10.16mm_Horizontal" V 7430 3500 50  0001 C CNN
 F 3 "~" H 7500 3500 50  0001 C CNN
 	1    7500 3500
@@
 F 0 "C1" H 4318 2296 50  0000 L CNN
 F 1 "22pF" H 4318 2205 50  0000 L CNN
-F 2 "" H 4238 2100 50  0001 C CNN
+F 2 "Capacitor_THT:CP_Radial_Tantal_D6.0mm_P5.00mm" H 4238 2100 50  0001 C CNN
 F 3 "~" H 4200 2250 50  0001 C CNN
 	1    4200 2250
@@
 F 0 "C2" H 4318 2896 50  0000 L CNN
 F 1 "22pF" H 4318 2805 50  0000 L CNN
-F 2 "" H 4238 2700 50  0001 C CNN
+F 2 "Capacitor_THT:CP_Radial_Tantal_D6.0mm_P5.00mm" H 4238 2700 50  0001 C CNN
 F 3 "~" H 4200 2850 50  0001 C CNN
 	1    4200 2850
@@
 F 0 "C3" H 3018 4946 50  0000 L CNN
 F 1 "10uF" H 3018 4855 50  0000 L CNN
-F 2 "" H 2938 4750 50  0001 C CNN
+F 2 "Capacitor_THT:CP_Radial_D10.0mm_P5.00mm" H 2938 4750 50  0001 C CNN
 F 3 "~" H 2900 4900 50  0001 C CNN
 	1    2900 4900
@@
 F 0 "R2" H 3680 4904 50  0000 R CNN
 F 1 "10k" H 3680 4995 50  0000 R CNN
-F 2 "" V 3680 4950 50  0001 C CNN
+F 2 "Resistor_THT:R_Axial_DIN0207_L6.3mm_D2.5mm_P10.16mm_Horizontal" V 3680 4950 50  0001 C CNN
 F 3 "~" H 3750 4950 50  0001 C CNN
 	1    3750 4950
@@
 F 0 "R3" H 3980 4904 50  0000 R CNN
 F 1 "10k" H 3980 4995 50  0000 R CNN
-F 2 "" V 3980 4950 50  0001 C CNN
+F 2 "Resistor_THT:R_Axial_DIN0207_L6.3mm_D2.5mm_P10.16mm_Horizontal" V 3980 4950 50  0001 C CNN
 F 3 "~" H 4050 4950 50  0001 C CNN
 	1    4050 4950
@@
 F 0 "R5" V 7707 3800 50  0000 C CNN
 F 1 "1k" V 7616 3800 50  0000 C CNN
-F 2 "" V 7430 3800 50  0001 C CNN
+F 2 "Resistor_THT:R_Axial_DIN0207_L6.3mm_D2.5mm_P10.16mm_Horizontal" V 7430 3800 50  0001 C CNN
 F 3 "~" H 7500 3800 50  0001 C CNN
 	1    7500 3800
@@
 F 0 "R6" V 7707 4100 50  0000 C CNN
 F 1 "1k" V 7616 4100 50  0000 C CNN
-F 2 "" V 7430 4100 50  0001 C CNN
+F 2 "Resistor_THT:R_Axial_DIN0207_L6.3mm_D2.5mm_P10.16mm_Horizontal" V 7430 4100 50  0001 C CNN
 F 3 "~" H 7500 4100 50  0001 C CNN
 	1    7500 4100
@@
 F 0 "R7" V 7707 4400 50  0000 C CNN
 F 1 "1k" V 7616 4400 50  0000 C CNN
-F 2 "" V 7430 4400 50  0001 C CNN
+F 2 "Resistor_THT:R_Axial_DIN0207_L6.3mm_D2.5mm_P10.16mm_Horizontal" V 7430 4400 50  0001 C CNN
 F 3 "~" H 7500 4400 50  0001 C CNN
 	1    7500 4400
@@
 Wire Wire Line
 	4450 4600 4450 5700
-Wire Wire Line
-	2850 3900 6350 3900
-Wire Wire Line
-	2850 4000 6350 4000
-Wire Wire Line
-	2850 4100 6250 4100
 Wire Wire Line
 	6250 3800 6250 3500
@@
 F 0 "INPUT_1" V 1950 7850 50  0000 C CNN
 F 1 "5v" V 2050 7750 50  0000 L CNN
-F 2 "" H 2100 7650 50  0001 C CNN
+F 2 "Connector_Pin:Pin_D1.3mm_L11.0mm" H 2100 7650 50  0001 C CNN
 F 3 "~" H 2100 7650 50  0001 C CNN
 	1    2100 7650
@@
 F 0 "INPUT_2" V 2550 7700 50  0000 L CNN
 F 1 "5v" V 2650 7750 50  0000 L CNN
-F 2 "" H 2700 7650 50  0001 C CNN
+F 2 "Connector_Pin:Pin_D1.3mm_L11.0mm" H 2700 7650 50  0001 C CNN
 F 3 "~" H 2700 7650 50  0001 C CNN
 	1    2700 7650
@@
 F 0 "OUTPUT_1" V 804 7562 50  0000 R CNN
 F 1 "5v" V 713 7562 50  0000 R CNN
-F 2 "" H 650 7650 50  0001 C CNN
+F 2 "Connector_Pin:Pin_D1.3mm_L11.0mm" H 650 7650 50  0001 C CNN
 F 3 "~" H 650 7650 50  0001 C CNN
 	1    650  7650
@@
 F 0 "OUTPUT_2" V 1354 7562 50  0000 R CNN
 F 1 "5v" V 1263 7562 50  0000 R CNN
-F 2 "" H 1200 7650 50  0001 C CNN
+F 2 "Connector_Pin:Pin_D1.3mm_L11.0mm" H 1200 7650 50  0001 C CNN
 F 3 "~" H 1200 7650 50  0001 C CNN
 	1    1200 7650
@@
 	2700 5700 4450 5700
 $Comp
-L Connector:Conn_01x01_Male OUTPUT_1
+L Connector:Conn_01x01_Male OUTPUT_3
 U 1 1 5F7B40CC
 P 10150 2650
-F 0 "OUTPUT_1" H 10122 2582 50  0000 R CNN
+F 0 "OUTPUT_3" H 10122 2582 50  0000 R CNN
 F 1 "5v" H 10122 2673 50  0000 R CNN
-F 2 "" H 10150 2650 50  0001 C CNN
+F 2 "Connector_Pin:Pin_D1.3mm_L11.0mm" H 10150 2650 50  0001 C CNN
 F 3 "~" H 10150 2650 50  0001 C CNN
 	1    10150 2650
@@
 $EndComp
 $Comp
-L Connector:Conn_01x01_Male OUTPUT_2
+L Connector:Conn_01x01_Male OUTPUT_4
 U 1 1 5F7B583C
 P 10150 3400
-F 0 "OUTPUT_2" H 10122 3332 50  0000 R CNN
+F 0 "OUTPUT_4" H 10122 3332 50  0000 R CNN
 F 1 "5v" H 10122 3423 50  0000 R CNN
-F 2 "" H 10150 3400 50  0001 C CNN
+F 2 "Connector_Pin:Pin_D1.3mm_L11.0mm" H 10150 3400 50  0001 C CNN
 F 3 "~" H 10150 3400 50  0001 C CNN
 	1    10150 3400
@@
 $EndComp
 $Comp
-L Connector:Conn_01x01_Male OUTPUT_3
+L Connector:Conn_01x01_Male OUTPUT_5
 U 1 1 5F7B59E6
 P 10150 4500
-F 0 "OUTPUT_3" H 10122 4432 50  0000 R CNN
+F 0 "OUTPUT_5" H 10122 4432 50  0000 R CNN
 F 1 "5v" H 10122 4523 50  0000 R CNN
-F 2 "" H 10150 4500 50  0001 C CNN
+F 2 "Connector_Pin:Pin_D1.3mm_L11.0mm" H 10150 4500 50  0001 C CNN
 F 3 "~" H 10150 4500 50  0001 C CNN
 	1    10150 4500
@@
 $EndComp
 $Comp
-L Connector:Conn_01x01_Male OUTPUT_4
+L Connector:Conn_01x01_Male OUTPUT_6
 U 1 1 5F7B603D
 P 10150 5250
-F 0 "OUTPUT_4" H 10122 5182 50  0000 R CNN
+F 0 "OUTPUT_6" H 10122 5182 50  0000 R CNN
 F 1 "5v" H 10122 5273 50  0000 R CNN
-F 2 "" H 10150 5250 50  0001 C CNN
+F 2 "Connector_Pin:Pin_D1.3mm_L11.0mm" H 10150 5250 50  0001 C CNN
 F 3 "~" H 10150 5250 50  0001 C CNN
 	1    10150 5250
@@
 F 0 "GND_4" H 10178 5476 50  0000 L CNN
 F 1 "5v" H 10178 5385 50  0000 L CNN
-F 2 "" H 10150 5450 50  0001 C CNN
+F 2 "Connector_Pin:Pin_D1.3mm_L11.0mm" H 10150 5450 50  0001 C CNN
 F 3 "~" H 10150 5450 50  0001 C CNN
 	1    10150 5450
@@
 F 0 "GND_3" H 10178 4726 50  0000 L CNN
 F 1 "5v" H 10178 4635 50  0000 L CNN
-F 2 "" H 10150 4700 50  0001 C CNN
+F 2 "Connector_Pin:Pin_D1.3mm_L11.0mm" H 10150 4700 50  0001 C CNN
 F 3 "~" H 10150 4700 50  0001 C CNN
 	1    10150 4700
@@
 F 0 "GND_2" H 10178 3626 50  0000 L CNN
 F 1 "5v" H 10178 3535 50  0000 L CNN
-F 2 "" H 10150 3600 50  0001 C CNN
+F 2 "Connector_Pin:Pin_D1.3mm_L11.0mm" H 10150 3600 50  0001 C CNN
 F 3 "~" H 10150 3600 50  0001 C CNN
 	1    10150 3600
@@
 F 0 "GND_1" H 10178 2876 50  0000 L CNN
 F 1 "5v" H 10178 2785 50  0000 L CNN
-F 2 "" H 10150 2850 50  0001 C CNN
+F 2 "Connector_Pin:Pin_D1.3mm_L11.0mm" H 10150 2850 50  0001 C CNN
 F 3 "~" H 10150 2850 50  0001 C CNN
 	1    10150 2850
 	1    0    0    -1
 $EndComp
+Wire Wire Line
+	2700 2800 3600 2800
+Wire Wire Line
+	2700 2900 3500 2900
+Wire Wire Line
+	2700 3800 6250 3800
+Wire Wire Line
+	2700 3900 6350 3900
+Wire Wire Line
+	2700 4000 6350 4000
+Wire Wire Line
+	2700 4100 6250 4100
+Wire Wire Line
+	2100 4550 2100 4600
+Connection ~ 2100 4600
+Wire Wire Line
+	2100 4600 2100 5200
 $EndSCHEMATC
