File: schematics/magic-curtains/magic-curtains-full.sch (KiCad schematic (older format))
At the start: 24 parts

Commit message: Did a full version and one for the PCB (without external components)
Parts:
- removed GND_1, GND_2, GND_3, GND_4, INPUT_1, INPUT_2: 5v, symbol Connector:Conn_01x01_Female
- removed OUTPUT_1 (x2), OUTPUT_2 (x2), OUTPUT_3, OUTPUT_4: 5v, symbol Connector:Conn_01x01_Male
- added External1, External2, External3, External4: Vv, symbol Connector:Conn_01x01_Female
- added K? (x2): ADW11, Relay_THT:Relay_1P1T_NO_10x24x18.8mm_Panasonic_ADW11xxxxW_THT, symbol Relay:ADW11
- added OUT1, OUT2, OUT3, OUT4: 5v, symbol Connector:Conn_01x01_Female
- added U? (x4): S102S02, Package_SIP:SIP4_Sharp-SSR_P7.62mm_Straight, symbol Relay_SolidState:S102S02
Connections:
- wire segments 93 -> 107
Other:
- note added: "A0-A5"
- note added: "CRESTRON MPC-M5"
